File: carry53-pcb-r2.kicad_pcb (KiCad board)
At the start: 2 copper layers, 292 x 82 mm, 191 parts, among them J1 Conn_01x02, J2 Conn_01x03, SW1 TS-1187A-B-A-B, SW2 TS-1187A-B-A-B, U1 STM32F072CBT6, U2 XC6206P332MR

Commit message: haisen_hobo_dekita
Parts:
- removed the REF** at (15.0, 15.3)
- removed the REF** at (15.0, 89.7)
- removed the REF** at (299.5, 15.0)
- removed the REF** at (299.4, 89.6)
Other:
- outline, holes or cut-outs redrawn
Changed lines of the file:
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@@
     (tracks 1371)
     (zones 0)
-    (modules 191)
+    (modules 187)
     (nets 101)
   )
@@
   )
   (setup
-    (last_trace_width 0.381)
+    (last_trace_width 0.25)
     (user_trace_width 0.381)
     (trace_clearance 0.2)
@@
     (pad_to_mask_clearance 0.051)
     (solder_mask_min_width 0.25)
-    (aux_axis_origin 0 0)
+    (aux_axis_origin 14.2875 11.3875)
+    (grid_origin 12.1625 93.3875)
     (visible_elements FFFFFF7F)
     (pcbplotparams
@@
   )
   (module MountingHole:MountingHole_2.7mm_Pad (layer F.Cu)
-    (at 15.0495 15.3035)
-    (descr "Mounting Hole 2.7mm")
-    (tags "mounting hole 2.7mm")
-    (attr virtual)
-    (fp_text reference REF** (at 0 -3.7) (layer F.SilkS)
-      (effects (font (size 1 1) (thickness 0.15)))
-    )
-    (fp_text value MountingHole_2.7mm_Pad (at 0 3.7) (layer F.Fab)
-      (effects (font (size 1 1) (thickness 0.15)))
-    )
-    (fp_circle (center 0 0) (end 2.95 0) (layer F.CrtYd) (width 0.05))
-    (fp_circle (center 0 0) (end 2.7 0) (layer Cmts.User) (width 0.15))
-    (fp_text user %R (at 0.3 0) (layer F.Fab)
-      (effects (font (size 1 1) (thickness 0.15)))
-    )
-    (pad 1 thru_hole circle (at 0 0) (size 5 5) (drill 2.7) (layers *.Cu *.Mask))
-  )
-  (module MountingHole:MountingHole_2.7mm_Pad (layer F.Cu)
-    (at 15.0495 89.7255)
-    (descr "Mounting Hole 2.7mm")
-    (tags "mounting hole 2.7mm")
-    (attr virtual)
-    (fp_text reference REF** (at 0 -3.7) (layer F.SilkS)
-      (effects (font (size 1 1) (thickness 0.15)))
-    )
-    (fp_text value MountingHole_2.7mm_Pad (at 0 3.7) (layer F.Fab)
-      (effects (font (size 1 1) (thickness 0.15)))
-    )
-    (fp_text user %R (at 0.3 0) (layer F.Fab)
-      (effects (font (size 1 1) (thickness 0.15)))
-    )
-    (fp_circle (center 0 0) (end 2.7 0) (layer Cmts.User) (width 0.15))
-    (fp_circle (center 0 0) (end 2.95 0) (layer F.CrtYd) (width 0.05))
-    (pad 1 thru_hole circle (at 0 0) (size 5 5) (drill 2.7) (layers *.Cu *.Mask))
-  )
-  (module MountingHole:MountingHole_2.7mm_Pad (layer F.Cu)
-    (at 299.5295 15.0495)
-    (descr "Mounting Hole 2.7mm")
-    (tags "mounting hole 2.7mm")
-    (attr virtual)
-    (fp_text reference REF** (at 0 -3.7) (layer F.SilkS)
-      (effects (font (size 1 1) (thickness 0.15)))
-    )
-    (fp_text value MountingHole_2.7mm_Pad (at 0 3.7) (layer F.Fab)
-      (effects (font (size 1 1) (thickness 0.15)))
-    )
-    (fp_circle (center 0 0) (end 2.95 0) (layer F.CrtYd) (width 0.05))
-    (fp_circle (center 0 0) (end 2.7 0) (layer Cmts.User) (width 0.15))
-    (fp_text user %R (at 0.3 0) (layer F.Fab)
-      (effects (font (size 1 1) (thickness 0.15)))
-    )
-    (pad 1 thru_hole circle (at 0 0) (size 5 5) (drill 2.7) (layers *.Cu *.Mask))
-  )
-  (module MountingHole:MountingHole_2.7mm_Pad (layer F.Cu)
     (at 117.475 15.08125)
     (descr "Mounting Hole 2.7mm")
@@
   )
   (module MountingHole:MountingHole_2.7mm_Pad (layer F.Cu)
-    (at 299.4025 89.5985)
-    (descr "Mounting Hole 2.7mm")
-    (tags "mounting hole 2.7mm")
-    (attr virtual)
-    (fp_text reference REF** (at 0 -3.7) (layer F.SilkS)
-      (effects (font (size 1 1) (thickness 0.15)))
-    )
-    (fp_text value MountingHole_2.7mm_Pad (at 0 3.7) (layer F.Fab)
-      (effects (font (size 1 1) (thickness 0.15)))
-    )
-    (fp_circle (center 0 0) (end 2.95 0) (layer F.CrtYd) (width 0.05))
-    (fp_circle (center 0 0) (end 2.7 0) (layer Cmts.User) (width 0.15))
-    (fp_text user %R (at 0.3 0) (layer F.Fab)
-      (effects (font (size 1 1) (thickness 0.15)))
-    )
-    (pad 1 thru_hole circle (at 0 0) (size 5 5) (drill 2.7) (layers *.Cu *.Mask))
-  )
-  (module MountingHole:MountingHole_2.7mm_Pad (layer F.Cu)
     (at 258.2545 52.1335)
     (descr "Mounting Hole 2.7mm")
@@
     )
   )
-  (gr_arc (start 302.1625 12.3875) (end 303.1625 12.3875) (angle -90) (layer Edge.Cuts) (width 0.12))
-  (gr_arc (start 302.1625 92.3875) (end 302.1625 93.3875) (angle -90) (layer Edge.Cuts) (width 0.12))
-  (gr_arc (start 12.1625 92.3875) (end 11.1625 92.3875) (angle -90) (layer Edge.Cuts) (width 0.12))
-  (gr_arc (start 12.1625 12.3875) (end 12.1625 11.3875) (angle -90) (layer Edge.Cuts) (width 0.12))
+  (gr_arc (start 13.1625 91.3875) (end 11.1625 91.3875) (angle -90) (layer Edge.Cuts) (width 0.12))
+  (gr_arc (start 301.1625 91.3875) (end 301.1625 93.3875) (angle -90) (layer Edge.Cuts) (width 0.12))
+  (gr_arc (start 301.1625 13.3875) (end 303.1625 13.3875) (angle -90) (layer Edge.Cuts) (width 0.12))
+  (gr_arc (start 13.1625 13.3875) (end 13.1625 11.3875) (angle -90) (layer Edge.Cuts) (width 0.12))
   (dimension 3.125 (width 0.15) (layer Eco1.User)
     (gr_text "3.125 mm" (at 12.725 98.3875) (layer Eco1.User)
@@
     (arrow2b (pts (xy 14.2875 5.211261) (xy 15.414004 4.62484)))
   )
-  (gr_line (start 302.1625 11.3875) (end 12.1625 11.3875) (layer Edge.Cuts) (width 0.12))
-  (gr_line (start 303.1625 92.3875) (end 303.1625 12.3875) (layer Edge.Cuts) (width 0.12))
-  (gr_line (start 12.1625 93.3875) (end 302.1625 93.3875) (layer Edge.Cuts) (width 0.12))
-  (gr_line (start 11.1625 12.3875) (end 11.1625 92.3875) (layer Edge.Cuts) (width 0.12))
+  (gr_line (start 301.1625 11.3875) (end 13.1625 11.3875) (layer Edge.Cuts) (width 0.12))
+  (gr_line (start 303.1625 91.3875) (end 303.1625 13.3875) (layer Edge.Cuts) (width 0.12))
+  (gr_line (start 13.1625 93.3875) (end 301.1625 93.3875) (layer Edge.Cuts) (width 0.12))
+  (gr_line (start 11.1625 13.3875) (end 11.1625 91.3875) (layer Edge.Cuts) (width 0.12))
   (segment (start 38.8575 33.7545) (end 38.4175 33.3145) (width 0.25) (layer B.Cu) (net 1))
   (segment (start 40.351 33.7545) (end 38.8575 33.7545) (width 0.25) (layer B.Cu) (net 1))
