File: carry53-pcb.kicad_pcb (KiCad board)
At the start: 2 copper layers, 292 x 82 mm, 191 parts, among them J1 Conn_01x02, J2 Conn_01x03, SW1 TS-1187A-B-A-B, SW2 TS-1187A-B-A-B, U1 STM32F072CBT6, U2 XC6206P332MR

Commit message: hobo kansei minaoshi hituyou kana
Parts:
- removed the REF** at (15.0, 15.3)
- removed the REF** at (213.5, 89.7)
- removed the REF** at (117.5, 89.7)
- removed the REF** at (15.0, 89.7)
- removed the REF** at (299.5, 15.0)
- removed the REF** at (117.5, 15.1)
- removed the REF** at (213.5, 15.1)
- removed the REF** at (68.3, 52.4)
- removed the REF** at (299.4, 89.6)
- removed the REF** at (258.3, 52.1)
- removed the REF** at (166.7, 53.2)
- added REF**: MountingHole_2.2mm_M2, MountingHole:MountingHole_2.2mm_M2, F.Cu at (299.5, 15.0)
- added REF**: MountingHole_2.2mm_M2, MountingHole:MountingHole_2.2mm_M2, F.Cu at (214.3, 20.0)
- added REF**: MountingHole_2.2mm_M2, MountingHole:MountingHole_2.2mm_M2, F.Cu at (15.0, 15.3)
- added REF**: MountingHole_2.2mm_M2, MountingHole:MountingHole_2.2mm_M2, F.Cu at (68.3, 52.4)
- added REF**: MountingHole_2.2mm_M2, MountingHole:MountingHole_2.2mm_M2, F.Cu at (166.7, 52.4)
- added REF**: MountingHole_2.2mm_M2, MountingHole:MountingHole_2.2mm_M2, F.Cu at (258.3, 52.4)
- added REF**: MountingHole_2.2mm_M2, MountingHole:MountingHole_2.2mm_M2, F.Cu at (219.0, 84.2)
- added REF**: MountingHole_2.2mm_M2, MountingHole:MountingHole_2.2mm_M2, F.Cu at (114.3, 84.3)
- added REF**: MountingHole_2.2mm_M2, MountingHole:MountingHole_2.2mm_M2, F.Cu at (299.4, 89.6)
- added REF**: MountingHole_2.2mm_M2, MountingHole:MountingHole_2.2mm_M2, F.Cu at (119.1, 19.9)
- added REF**: MountingHole_2.2mm_M2, MountingHole:MountingHole_2.2mm_M2, F.Cu at (15.0, 89.7)
- moved J2 5.08 mm to (38.8, 16.0), turned to 0 degrees
- moved D10 0.27 mm to (214.3, 25.7)
- moved J1 0.07 mm to (41.5, 16.0)
Routing:
- net COL4: track 184.0 -> 204.2 mm
- net COL9: track 295.1 -> 311.4 mm
- net SWDIO: track 27.4 -> 20.8 mm
- net COL6: track 244.5 -> 250.9 mm
- net NRST: track 93.2 -> 98.2 mm
- net ROW3: track 448.3 -> 445.1 mm
- net Net-(D10-Pad2): track 14.1 -> 17.3 mm
- net Net-(D5-Pad2): track 14.7 -> 17.2 mm
- net COL11: track 343.5 -> 345.4 mm
- net COL8: track 295.4 -> 294.2 mm
- net COL3: track 162.7 -> 161.9 mm
Other:
- outline, holes or cut-outs redrawn
- board text added: "Carry53 v1.0"

Commit message: kansei de iiyone
Parts:
- moved D1 16.1 mm to (19.9, 19.8)
- moved C6 8.97 mm to (15.0, 56.5), turned to 0 degrees
- moved R1 5.24 mm to (15.0, 58.1), turned to 0 degrees
- moved D15 3.88 mm to (38.4, 48.7)
- moved F1 2.01 mm to (22.0, 40.1), turned to 180 degrees
- moved C7 1.18 mm to (26.3, 29.9)
- moved R2 1.15 mm to (23.1, 30.7), turned to 90 degrees
- moved R3 1.11 mm to (23.1, 36.1), turned to 270 degrees
- moved U2 1.06 mm to (29.5, 29.9), turned to 180 degrees
- moved ESD1 0.83 mm to (24.6, 34.6)
- moved ESD2 0.83 mm to (24.6, 32.1)
- moved C3 0.75 mm to (50.3, 32.7), turned to 90 degrees
- moved C8 0.59 mm to (32.6, 29.9)
- moved SW1 0.11 mm to (14.9, 51.5)
Routing:
- net ROW0: track 372.6 -> 396.6 mm
- net NRST: track 98.2 -> 113.2 mm, vias 3 -> 2
- net GND: track 195.4 -> 181.2 mm
- net Net-(R1-Pad1): track 62.9 -> 72.4 mm
- net ROW1: track 424.8 -> 417.8 mm
- net Net-(C7-Pad1): track 18.4 -> 12.8 mm
- net +3V3: track 154.1 -> 148.5 mm
- net Net-(D15-Pad2): track 22.1 -> 18.8 mm
- net Net-(F1-Pad2): track 16.5 -> 15.1 mm
- net Net-(D1-Pad2): track 10.2 -> 11.6 mm
- net Net-(R2-Pad1): track 4.64 -> 3.85 mm
- net COL1: track 137.6 -> 138.3 mm
- net Net-(R3-Pad1): track 4.84 -> 4.13 mm
- net ROW2: track 427.9 -> 427.1 mm
